File: cube.sch (KiCad schematic (older format))
At the start: 0 parts

Commit message: Add cube PCB design
Parts:
- added C? (x3): 0.1uF, symbol Device:C
- added CB? (x3), cb?: 1uF, symbol Device:C_Small
- added CX? (x2): 12pF, symbol Device:C_Small
- added R?: 470, symbol Device:R
- added R?: 10k, symbol Device:R
- added U?: AT86RF231-ZU, 32QN2_ATM, symbol zigbee:AT86RF231-ZU
- added U?: PIC18F47K40-I_P, PDIP40_P_MCH, symbol pic18f47:PIC18F47K40-I_P
- added XTAL?: CX-4025 16Mhz, symbol Device:Crystal
Connections:
- new net: CB?.2, U?.29 (AVDD)
- new net: U?.13 (DVDD), U?.14 (DVDD), cb?.1
- new net: CX?.2, U?.25 (XTAL2), XTAL?.2
- new net: CX?.1, U?.26 (XTAL1), XTAL?.1
- new net: R?.1, U?.1 (*MCLR/VPP/RE3)
- new net: C?.2, R?.2, R?.2
- new net +3V3: C?.1, C?.2, CB?.1, CB?.1, R?.1, U?.11 (VDD), U?.15 (DEVDD), U?.28 (EVDD), U?.32 (VDD)
- new net GND: C?.1, C?.1, C?.2, CB?.1, CB?.2, CB?.2, CX?.1, CX?.2, U?.1 (DIG3), U?.10 (DIG2), U?.12 (DVSS), U?.12 (VSS), U?.16 (DVSS), U?.18 (DVSS), U?.2 (DIG4), U?.21 (DVSS), U?.27 (AVSS), U?.3 (AVSS), U?.30 (AVSS), U?.31 (AVSS), U?.31 (VSS), U?.32 (AVSS), U?.33, U?.6 (AVSS), U?.7 (DVSS), U?.9 (DIG1), cb?.2
- new net IRQ_ZGB: U?.24 (IRQ), U?.36 (RB3)
- new net RESET_ZGB: U?.38 (RB6), U?.8 (*RST)
- new net SLP_TR: U?.11 (SLP_TR), U?.37 (RB4)
- new net SPI_CLK: U?.18 (RC3), U?.19 (SCLK)
- new net SPI_CS1: U?.23 (*SEL), U?.7 (RA5)
- new net SPI_MISO: U?.20 (MISO), U?.23 (RC4)
- new net SPI_MOSI: U?.22 (MOSI), U?.22 (RD3)
- no-connect marks 0 -> 1
