File: hub.sch (KiCad schematic (older format))
At the start: 14 parts

Commit message: Edit HUB PCB
Parts:
- removed R?: 680Ω, symbol Device:R_Small
- added R?: 680, symbol Device:R
- gave numbers to parts that had none: 5
Connections:
- wire segments 135 -> 133
Changed lines of the file:
@@
 	1    0    0    -1
 $EndComp
-$Comp
-L power:GND #PWR?
-U 1 1 6089C046
-P 9050 2900
-F 0 "#PWR?" H 9050 2650 50  0001 C CNN
-F 1 "GND" V 9055 2772 50  0000 R CNN
-F 2 "" H 9050 2900 50  0001 C CNN
-F 3 "" H 9050 2900 50  0001 C CNN
-	1    9050 2900
-	0    -1   -1   0
-$EndComp
-Wire Wire Line
-	8950 2900 9050 2900
 Text Notes 6300 1100 0    354  ~ 0
 WI-FI MODULE
 Wire Wire Line
 	9350 3050 9750 3050
-Text GLabel 9350 3050 0    50   Input ~ 0
-RESET
 Wire Wire Line
 	13350 3050 12950 3050
@@
 CLKM
 $Comp
-L Device:C_Small C?
+L Device:C_Small c
 U 1 1 607FC9EB
 P 6250 10050
-F 0 "C?" H 6342 10096 50  0000 L CNN
+F 0 "c" H 6342 10096 50  0001 L CNN
 F 1 "2.2pF" H 6342 10005 50  0000 L CNN
 F 2 "" H 6250 10050 50  0001 C CNN
@@
 $EndComp
 $Comp
-L Device:C_Small CX?
+L Device:C_Small CX2
 U 1 1 607FC9C8
 P 6450 9350
-F 0 "CX?" V 6655 9350 39  0000 C CNN
+F 0 "CX2" V 6655 9350 39  0000 C CNN
 F 1 "12pF" V 6580 9350 39  0000 C CNN
 F 2 "" H 6450 9350 50  0001 C CNN
@@
 $EndComp
 $Comp
-L Device:C_Small CX?
+L Device:C_Small CX1
 U 1 1 607FC9C2
 P 6450 8750
-F 0 "CX?" V 6245 8750 39  0000 C CNN
+F 0 "CX1" V 6245 8750 39  0000 C CNN
 F 1 "12pF" V 6320 8750 39  0000 C CNN
 F 2 "" H 6450 8750 50  0001 C CNN
@@
 U 1 1 607FC9BC
 P 6250 8400
-F 0 "CB?" V 6021 8400 50  0000 C CNN
+F 0 "CB?" V 6021 8400 50  0001 C CNN
 F 1 "1uF" V 6112 8400 50  0000 C CNN
 F 2 "" H 6250 8400 50  0001 C CNN
@@
 	6150 8800 6150 8400
 $Comp
-L Device:Crystal XTAL?
+L Device:Crystal XTAL
 U 1 1 607FC996
 P 6300 9050
-F 0 "XTAL?" V 6262 9181 39  0000 L CNN
+F 0 "XTAL" V 6262 9181 39  0000 L CNN
 F 1 "CX-4025 16Mhz" V 6337 9181 39  0000 L CNN
 F 2 "" H 6300 9050 50  0001 C CNN
@@
 	0    -1   -1   0
 $EndComp
-Connection ~ 6250 9900
 $Comp
 L power:GND #PWR?
@@
 U 1 1 607FC9B6
 P 5400 8700
-F 0 "CB?" V 5171 8700 50  0000 C CNN
+F 0 "CB?" V 5171 8700 50  0001 C CNN
 F 1 "1uF" V 5262 8700 50  0000 C CNN
 F 2 "" H 5400 8700 50  0001 C CNN
@@
 SCLK
 $Comp
-L Device:R_Small R?
-U 1 1 607FC9F1
-P 5750 9900
-F 0 "R?" V 5554 9900 50  0000 C CNN
-F 1 "680Ω" V 5645 9900 50  0000 C CNN
-F 2 "" H 5750 9900 50  0001 C CNN
-F 3 "~" H 5750 9900 50  0001 C CNN
-	1    5750 9900
-	0    1    1    0
-$EndComp
-Wire Wire Line
-	5150 9900 5650 9900
-Wire Wire Line
-	5650 9900 5850 9900
-Connection ~ 5650 9900
-Wire Wire Line
-	5850 9900 6250 9900
-Connection ~ 5850 9900
-$Comp
 L power:GND #PWR?
 U 1 1 607FCA07
@@
 $EndComp
 $Comp
-L Device:C_Small CB?
+L Device:C_Small cb
 U 1 1 607FCA3A
 P 2600 9400
-F 0 "CB?" V 2371 9400 50  0000 C CNN
+F 0 "cb" V 2371 9400 50  0001 C CNN
 F 1 "1uF" V 2462 9400 50  0000 C CNN
 F 2 "" H 2600 9400 50  0001 C CNN
@@
 U 1 1 607FCA54
 P 2600 9700
-F 0 "CB?" V 2829 9700 50  0000 C CNN
+F 0 "CB?" V 2829 9700 50  0001 C CNN
 F 1 "1uF" V 2738 9700 50  0000 C CNN
 F 2 "" H 2600 9700 50  0001 C CNN
@@
 	1    0    0    -1
 $EndComp
+Text GLabel 9350 3050 0    50   Input ~ 0
+RESET
+$Comp
+L Device:R R?
+U 1 1 6082C987
+P 5650 9900
+F 0 "R?" V 5443 9900 50  0001 C CNN
+F 1 "680" V 5535 9900 50  0000 C CNN
+F 2 "" V 5580 9900 50  0001 C CNN
+F 3 "~" H 5650 9900 50  0001 C CNN
+	1    5650 9900
+	0    1    1    0
+$EndComp
+Wire Wire Line
+	5150 9900 5500 9900
+Wire Wire Line
+	5800 9900 6250 9900
+Connection ~ 6250 9900
 $EndSCHEMATC

Commit message: Edit hub pcb
Parts:
- removed HUB_MCU: PIC32MX575F512H, symbol MCU_Microchip_PIC32:PIC32MX575F512H
- added C?, CBp (x3): 0.1uF, symbol Device:C
- added R?: 10, symbol Device:R
- added U?: PIC32MX575F512H-80I_PT, TQFP64_10x10MC_MCH, symbol pic32mx575:PIC32MX575F512H-80I_PT
Connections:
- net GND: now also C?.1
- new net: CBp.2, R?.1, U?.10 (VDD)
- new net: CBp.1, R?.2, U?.19 (AVDD)
- new net: CBp.2, U?.20 (AVSS)
- new net: CBp.1, U?.25 (VSS)
- new net: CBp.2, U?.26 (VDD)
- new net: C?.2, U?.38 (VDD)
- new net: C?.1, U?.41 (VSS)
- new net: CBp.1, U?.9 (VSS)
Other:
- moved on the sheet: C?, CX1, CX2, U?, XTAL

Commit message: Finish hub pcb schema
Parts:
- removed CBp (x2): 0.1uF, symbol Device:C
- removed R?: 680, symbol Device:R
- removed R?: 10, symbol Device:R
- removed c: 2.2pF, symbol Device:C_Small
- added C, C?, CBp (x2): 0.1uF, symbol Device:C
- added C?: 0.25pF, symbol Device:C
- added R?: 10, symbol Device:R
- added R?: R, symbol Device:R
- added R?: R1, symbol Device:R
Connections:
- net GND is gone; now on net +3V3: C?.1, CB?.1, CB?.2, CB?.2, CX1.2, CX2.1, R?.2, U?.1 (DIG3), U?.10 (DIG2), U?.12 (DVSS), U?.16 (DVSS), U?.18 (DVSS), U?.2 (DIG4), U?.21 (DVSS), U?.27 (AVSS), U?.3 (AVSS), U?.30 (AVSS), U?.31 (AVSS), U?.32 (AVSS), U?.33, U?.6 (AVSS), U?.7 (DVSS), U?.9 (DIG1), WiFi.1 (GND), WiFi.11 (GND), WiFi.21 (GND), WiFi.26 (SDIO_DAT2/HIF_SEL), WiFi.35 (GND), WiFi.36 (GND), WiFi.39 (RESERVE_1), WiFi.4 (GND), WiFi.41 (GND), WiFi.42 (GND), WiFi.43 (GND), WiFi.44 (GND), WiFi.45 (GND), WiFi.46 (GND), WiFi.48 (GND), WiFi.49 (GND), WiFi.5 (GND), WiFi.50 (GND), WiFi.51 (GND), WiFi.52 (GND), WiFi.53 (GND), WiFi.54 (GND), WiFi.55 (GND), WiFi.56 (GND), WiFi.57 (GND), WiFi.58 (GND), WiFi.6 (GND), WiFi.7 (GND), WiFi.8 (GND), cb.2
- net IRQ is gone; now on net IRQ_ZGB: U?.24 (IRQ)
- net RESET is gone; now on net RESET_WF: WiFi.12 (RESETN)
- net RST is gone; now on net RESET_ZGB: U?.8 (*RST)
- net SCLK is gone; now on net SPI_CLK: U?.19 (SCLK)
- net SEL is gone; now on net SPI_CS1: U?.23 (*SEL)
- net WIRQ is gone; now on net IRQ_WF: WiFi.19 (GPIO/WIRQ)
- net +3V3: now also C?.1, C?.2, CBp.1, U?.20 (AVSS), U?.26 (VDD), U?.38 (VDD), U?.41 (VSS), U?.57 (VDD), U?.9 (VSS), C.1, C?.1, C?.1, C?.2, CBp.1, CBp.1, R?.1
- net LP_CLK: now also U?.48 (SOSCO/T1CK/CN0/RC14)
- net SLP_TR: now also U?.2 (PMD6/RE6)
- net SPI_CLK: now also U?.49 (SCK1A/U1BTX/*U1ARTS/OC2/RD1)
- net SPI_CS2: now also U?.42 (RTCC/IC1/INT1/RD8)
- net SPI_IRQ: now also U?.52 (OC5/IC5/PMWR/CN13/RD4)
- net SPI_MISO: now also U?.50 (SDA1A/SDI1A/U1ARX/OC3/RD2)
- net SPI_MOSI: now also U?.51 (SCL1A/SDO1A/U1ATX/OC4/RD3)
- net WUP: now also U?.63 (PMD3/RE3)
- net RESET_ZGB: now reaches U?.1 (PMD5/RE5)
- net at CBp.2, U?.10 (VDD): now also R?.1
- net at U?.19 (AVDD): now also CBp.2, R?.2
- net at U?.25 (VSS): now also CBp.2
- net IRQ_ZGB: now reaches U?.3 (PMD7/RE7)
- net SPI_CS1: now reaches U?.43 (*SS1A/U1BRX/*U1ACTS/SDA1/IC2/INT2/RD9)
- net at U?.56 (VCAP/VCORE): now also C?.2
- net RESET_WF: now reaches U?.62 (PMD2/RE2)
- net IRQ_WF: now reaches U?.64 (PMD4/RE4)
- net at U?.7 (*MCLR): now also R?.2
- new net: C.2, R?.1, R?.2
Other:
- moved on the sheet: CBp
