File: Cube/cube.sch (KiCad schematic (older format))
At the start: 22 parts

Commit message: Add minor changes
Parts:
- added R?: 330, symbol Device:R
Connections:
- net LED_DATA: now also R?.1; no longer J?.2 (Pin_2)
- new net: J?.2 (Pin_2), R?.2
Changed lines of the file:
@@
 L Connector:Conn_01x03_Male J?
 U 1 1 607FB043
-P 8050 2550
-F 0 "J?" H 8158 2831 50  0001 C CNN
-F 1 "Conn_01x03_Male" H 8158 2739 50  0001 C CNN
-F 2 "" H 8050 2550 50  0001 C CNN
-F 3 "~" H 8050 2550 50  0001 C CNN
-	1    8050 2550
+P 8250 2550
+F 0 "J?" H 8358 2831 50  0001 C CNN
+F 1 "Conn_01x03_Male" H 8358 2739 50  0001 C CNN
+F 2 "" H 8250 2550 50  0001 C CNN
+F 3 "~" H 8250 2550 50  0001 C CNN
+	1    8250 2550
 	-1   0    0    -1
 $EndComp
 Wire Wire Line
-	7850 2650 7600 2650
+	8050 2650 7800 2650
 $Comp
 L power:+5V #PWR?
 U 1 1 6080BDAA
-P 7600 2650
-F 0 "#PWR?" H 7600 2500 50  0001 C CNN
-F 1 "+5V" V 7615 2778 50  0000 L CNN
-F 2 "" H 7600 2650 50  0001 C CNN
-F 3 "" H 7600 2650 50  0001 C CNN
-	1    7600 2650
+P 7800 2650
+F 0 "#PWR?" H 7800 2500 50  0001 C CNN
+F 1 "+5V" V 7815 2778 50  0000 L CNN
+F 2 "" H 7800 2650 50  0001 C CNN
+F 3 "" H 7800 2650 50  0001 C CNN
+	1    7800 2650
 	0    -1   -1   0
 $EndComp
@@
 L power:GND #PWR?
 U 1 1 6080D5D3
-P 7600 2450
-F 0 "#PWR?" H 7600 2200 50  0001 C CNN
-F 1 "GND" V 7605 2322 50  0000 R CNN
-F 2 "" H 7600 2450 50  0001 C CNN
-F 3 "" H 7600 2450 50  0001 C CNN
-	1    7600 2450
+P 7800 2450
+F 0 "#PWR?" H 7800 2200 50  0001 C CNN
+F 1 "GND" V 7805 2322 50  0000 R CNN
+F 2 "" H 7800 2450 50  0001 C CNN
+F 3 "" H 7800 2450 50  0001 C CNN
+	1    7800 2450
 	0    1    1    0
 $EndComp
 Wire Wire Line
-	7600 2450 7850 2450
-Wire Wire Line
-	7850 2550 7550 2550
-Text GLabel 7550 2550 0    50   Input ~ 0
+	7800 2450 8050 2450
+Text GLabel 7100 2550 0    50   Input ~ 0
 LED_DATA
 Text GLabel 1400 1600 0    50   Output ~ 0
@@
 Wire Wire Line
 	1750 1600 1400 1600
+$Comp
+L Device:R R?
+U 1 1 607F2183
+P 7400 2550
+F 0 "R?" H 7470 2596 50  0001 L CNN
+F 1 "330" V 7470 2472 50  0000 L CNN
+F 2 "" V 7330 2550 50  0001 C CNN
+F 3 "~" H 7400 2550 50  0001 C CNN
+	1    7400 2550
+	0    -1   -1   0
+$EndComp
+Wire Wire Line
+	7550 2550 8050 2550
+Wire Wire Line
+	7100 2550 7250 2550
+Text Label 8250 2450 0    50   ~ 0
+GND
+Text Label 8250 2650 0    50   ~ 0
+5V
+Text Label 8250 2550 0    50   ~ 0
+DATA
 $EndSCHEMATC
