File: Hub/hub.sch (KiCad schematic (older format))
At the start: 22 parts

Commit message: Update
Zigbee update:
- Added custom made symbol: SMD Balun - 2450FB15L0001E
- Added Antenna - Ceramic chip: W3043

Note: There might be a missing capacitor in the communication between the antenna to the Balun - some circuit reference does have it some doesn't
Parts:
- added B?: 2450FB15L0001E, symbol Balun:2450FB15L0001E
- added C1, C2, C3: 22pF, symbol Device:C_Small
- added W3043: 2.4GHz, symbol Device:Antenna
- U?: symbol zigbee:AT86RF231-ZU -> hub-rescue:AT86RF231-ZU-zigbee
- U?: symbol pic32mx575:PIC32MX575F512H-80I_PT -> hub-rescue:PIC32MX575F512H-80I_PT-pic32mx575
- WiFi: symbol 2021-04-18_17-18-12:WFM200S022XNA2 -> hub-rescue:WFM200S022XNA2-2021-04-18_17-18-12
Connections:
- wire segments 186 -> 203
Changed lines of the file:
@@
 HUB MCU
 $Comp
-L zigbee:AT86RF231-ZU U?
+L hub-rescue:AT86RF231-ZU-zigbee U?
 U 1 1 607D7BD3
 P 3250 11650
@@
 $EndComp
 $Comp
-L pic32mx575:PIC32MX575F512H-80I_PT U?
+L hub-rescue:PIC32MX575F512H-80I_PT-pic32mx575 U?
 U 1 1 6089B15F
 P 6700 2950
@@
 	13950 11250 13550 11250
 $Comp
-L 2021-04-18_17-18-12:WFM200S022XNA2 WiFi
+L hub-rescue:WFM200S022XNA2-2021-04-18_17-18-12 WiFi
 U 1 1 607CE80D
 P 13950 11250
@@
 Connection ~ 6100 4650
 Connection ~ 6100 4950
+$Comp
+L power:GND #PWR?
+U 1 1 607F320D
+P 1900 12650
+F 0 "#PWR?" H 1900 12400 50  0001 C CNN
+F 1 "GND" H 1905 12477 50  0000 C CNN
+F 2 "" H 1900 12650 50  0001 C CNN
+F 3 "" H 1900 12650 50  0001 C CNN
+	1    1900 12650
+	1    0    0    -1
+$EndComp
+$Comp
+L power:GND #PWR?
+U 1 1 607F3ACA
+P 1850 11700
+F 0 "#PWR?" H 1850 11450 50  0001 C CNN
+F 1 "GND" H 1855 11527 50  0000 C CNN
+F 2 "" H 1850 11700 50  0001 C CNN
+F 3 "" H 1850 11700 50  0001 C CNN
+	1    1850 11700
+	-1   0    0    1
+$EndComp
+$Comp
+L Device:C_Small C3
+U 1 1 607F44F6
+P 1900 12450
+F 0 "C3" H 1992 12488 39  0000 L CNN
+F 1 "22pF" H 1992 12413 39  0000 L CNN
+F 2 "" H 1900 12450 50  0001 C CNN
+F 3 "~" H 1900 12450 50  0001 C CNN
+	1    1900 12450
+	-1   0    0    1
+$EndComp
+$Comp
+L Device:C_Small C2
+U 1 1 607F514A
+P 2450 12250
+F 0 "C2" H 2542 12288 39  0000 L CNN
+F 1 "22pF" H 2542 12213 39  0000 L CNN
+F 2 "" H 2450 12250 50  0001 C CNN
+F 3 "~" H 2450 12250 50  0001 C CNN
+	1    2450 12250
+	0    1    1    0
+$EndComp
+$Comp
+L Device:C_Small C1
+U 1 1 607F63C6
+P 2450 11800
+F 0 "C1" H 2542 11838 39  0000 L CNN
+F 1 "22pF" H 2542 11763 39  0000 L CNN
+F 2 "" H 2450 11800 50  0001 C CNN
+F 3 "~" H 2450 11800 50  0001 C CNN
+	1    2450 11800
+	0    -1   -1   0
+$EndComp
+$Comp
+L Device:Antenna W3043
+U 1 1 607F6DE5
+P 1250 12300
+F 0 "W3043" H 1330 12281 39  0000 L CNN
+F 1 "2.4GHz" H 1330 12206 39  0000 L CNN
+F 2 "" H 1250 12300 50  0001 C CNN
+F 3 "~" H 1250 12300 50  0001 C CNN
+	1    1250 12300
+	0    -1   -1   0
+$EndComp
+$Comp
+L Balun:2450FB15L0001E B?
+U 1 1 607F83DB
+P 2550 12200
+F 0 "B?" V 2751 12622 50  0000 R CNN
+F 1 "2450FB15L0001E" V 2660 12622 50  0000 R CNN
+F 2 "" H 2700 13050 50  0001 C CNN
+F 3 "https://www.johansontechnology.com/datasheets/2450FB15L0001/2450FB15L0001.pdf" H 2700 13050 50  0001 C CNN
+	1    2550 12200
+	0    -1   -1   0
+$EndComp
+Wire Wire Line
+	1800 11900 1800 11750
+Wire Wire Line
+	1800 11750 1850 11750
+Wire Wire Line
+	1850 11750 1850 11700
+Wire Wire Line
+	1850 11750 1900 11750
+Wire Wire Line
+	1900 11750 1900 11900
+Connection ~ 1850 11750
+Wire Wire Line
+	2000 11900 2000 11800
+Wire Wire Line
+	2000 11800 2350 11800
+Wire Wire Line
+	2550 11800 2550 11950
+Wire Wire Line
+	2550 11950 3250 11950
+Wire Wire Line
+	2000 12150 2000 12250
+Wire Wire Line
+	2000 12250 2350 12250
+Wire Wire Line
+	2550 12250 2550 12050
+Wire Wire Line
+	2550 12050 3250 12050
+Wire Wire Line
+	1900 12550 1900 12650
+Wire Wire Line
+	1900 12350 1900 12150
+Wire Wire Line
+	1800 12150 1800 12300
+Wire Wire Line
+	1800 12300 1450 12300
 $EndSCHEMATC

Commit message: Add motor to the cube schematics
Other:
- moved on the sheet: C1, C2, C3, CX1, CX2, U?, W3043, XTAL

Commit message: Add power supply changes
Parts:
- added C? (x2): 100nF, Capacitor_SMD:C_0402_1005Metric, symbol Device:C
- added C?: 22µF, Capacitor_SMD:C_0402_1005Metric, symbol Device:C
- added C?: 10µF, Capacitor_SMD:C_0402_1005Metric, symbol Device:C
- added J?: Conn_01x01_Male, Connector_Pin:Pin_D0.7mm_L6.5mm_W1.8mm_FlatFork, symbol Connector:Conn_01x01_Male
- added J?: Barrel_Jack, symbol Connector:Barrel_Jack
- added L?: 4.7µH, Inductor_SMD:L_0402_1005Metric, symbol Device:L
- added R?: 30.9kΩ, Resistor_SMD:R_0402_1005Metric, symbol Device:R
- added R?: 10kΩ, Resistor_SMD:R_0402_1005Metric, symbol Device:R
- added R?: 30Ω, Resistor_SMD:R_0402_1005Metric, symbol Device:R
- added R?: 16.5k, Resistor_SMD:R_0402_1005Metric, symbol Device:R
- added R?: 13.7k, Resistor_SMD:R_0402_1005Metric, symbol Device:R
- added U?: TPS56339DDC, Package_TO_SOT_SMD:SOT-23-6, symbol Regulator_Switching:TPS56339DDC
Connections:
- net labels added: VCC
- wire segments 203 -> 247
- no-connect marks 14 -> 58
Other:
- note added: "3.3V, 1.8V out"
- note added: "BARREL JACK"
- moved on the sheet: C, C1, C2, C3, CBp, CBp?, CX1, CX2, U?, W3043, XTAL

Commit message: added both voltages to the hub
Parts:
- removed C? (x2): 100nF, Capacitor_SMD:C_0402_1005Metric, symbol Device:C
- removed C?: 22µF, Capacitor_SMD:C_0402_1005Metric, symbol Device:C
- removed C?: 10µF, Capacitor_SMD:C_0402_1005Metric, symbol Device:C
- removed J?: Conn_01x01_Male, Connector_Pin:Pin_D0.7mm_L6.5mm_W1.8mm_FlatFork, symbol Connector:Conn_01x01_Male
- removed L?: 4.7µH, Inductor_SMD:L_0402_1005Metric, symbol Device:L
- removed R?: 30.9kΩ, Resistor_SMD:R_0402_1005Metric, symbol Device:R
- removed R?: 10kΩ, Resistor_SMD:R_0402_1005Metric, symbol Device:R
- removed R?: 30Ω, Resistor_SMD:R_0402_1005Metric, symbol Device:R
- removed R?: 16.5k, Resistor_SMD:R_0402_1005Metric, symbol Device:R
- removed R?: 13.7k, Resistor_SMD:R_0402_1005Metric, symbol Device:R
- removed U?: TPS56339DDC, Package_TO_SOT_SMD:SOT-23-6, symbol Regulator_Switching:TPS56339DDC
- added C? (x4): 100nF, Capacitor_SMD:C_0402_1005Metric, symbol Device:C
- added C? (x2): 22µF, Capacitor_SMD:C_0402_1005Metric, symbol Device:C
- added C? (x2): 10µF, Capacitor_SMD:C_0402_1005Metric, symbol Device:C
- added L?: 2.2µH, Inductor_SMD:L_0402_1005Metric, symbol Device:L
- added L?: 4.7µH, Inductor_SMD:L_0402_1005Metric, symbol Device:L
- added R?: 12.4kΩ, Resistor_SMD:R_0402_1005Metric, symbol Device:R
- added R? (x2): 10kΩ, Resistor_SMD:R_0402_1005Metric, symbol Device:R
- added R? (x2): 30Ω, Resistor_SMD:R_0402_1005Metric, symbol Device:R
- added R?: 30.9kΩ, Resistor_SMD:R_0402_1005Metric, symbol Device:R
- added U? (x2): TPS56339DDC, Package_TO_SOT_SMD:SOT-23-6, symbol Regulator_Switching:TPS56339DDC
Connections:
- wire segments 247 -> 269
- no-connect marks 58 -> 59

Commit message: Add programmable connectors
Parts:
- removed C: 0.1uF, symbol Device:C
- removed R?: 470, symbol Device:R
- added J?: Conn_01x06_Male, symbol Connector:Conn_01x06_Male
- R?: value 10k -> 1k
Connections:
- net labels added: MCLR, PGC, PGD
- wire segments 269 -> 273
- no-connect marks 59 -> 55
Other:
- note added: "PICKIT CONNECTOR"
- moved on the sheet: C?, CBp, CBp?, J?, L?, R?, U?

Commit message: hub pcb stuck
Parts:
- removed B?: 2450FB15L0001E, symbol Balun:2450FB15L0001E
- added B1: 2450FB15L0001E-Balun, RF_Converter:Balun_Johanson_1.6x0.8mm, symbol hub-rescue:2450FB15L0001E-Balun
- C1, C2, C3, CX1, CX2: footprint (none) -> Capacitor_SMD:C_0603_1608Metric
- C10, C11, C12, C14, C15, C4, C5, C9: renamed from C?; footprint Capacitor_SMD:C_0402_1005Metric -> Capacitor_SMD:C_0603_1608Metric
- C13, C6, C7, C8: renamed from C?; footprint (none) -> Capacitor_SMD:C_0603_1608Metric
- CB1, CB2, CB3: renamed from CB?; footprint (none) -> Capacitor_SMD:C_0603_1608Metric
- CBp1: renamed from CBp; footprint (none) -> Capacitor_SMD:C_0603_1608Metric
- CBp2, CBp3: renamed from CBp?; footprint (none) -> Capacitor_SMD:C_0603_1608Metric
- J1: renamed from J?; footprint (none) -> Connector_BarrelJack:BarrelJack_CUI_PJ-063AH_Horizontal
- J2: renamed from J?; footprint (none) -> Connector_PinHeader_1.00mm:PinHeader_1x06_P1.00mm_Vertical
- L1, L2: renamed from L?; footprint Inductor_SMD:L_0402_1005Metric -> Inductor_SMD:L_0603_1608Metric
- R1, R2: renamed from R?; footprint (none) -> Resistor_SMD:R_0603_1608Metric
- R3, R4, R5, R6, R7, R8: renamed from R?; footprint Resistor_SMD:R_0402_1005Metric -> Resistor_SMD:R_0603_1608Metric
- RR1: renamed from r; footprint (none) -> Resistor_SMD:R_0603_1608Metric
- U1: renamed from U?; footprint TQFP64_10x10MC_MCH -> MCU_HUB:PIC32MX575F512H-80I&slash_PT
- U2: renamed from U?; footprint 32QN2_ATM -> ZBEE:AT86RF231-ZU
- W3043: footprint (none) -> RF_Antenna:Texas_SWRA117D_2.4GHz_Left
- WiFi1: renamed from WiFi; footprint QFN_S022XNA2_SIL -> WIFI:WFM200S022XNA2
- XTAL1: renamed from XTAL; footprint (none) -> Crystal:Crystal_SMD_MicroCrystal_CC4V-T1A-2Pin_5.0x1.9mm
- cb1: renamed from cb; footprint (none) -> Capacitor_SMD:C_0603_1608Metric
- gave numbers to parts that had none: 2
